Commit message: moved base_body joint outside

File: urdf/belt_robot.urdf (robot description, URDF)
Before this commit: robot robot, 2 links, 0 joints
Links:
- added link gripper_left; visual mesh filename=package://robotarm_description/meshes/belt_arm_ros_gripper_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
- added link gripper_right; visual mesh filename=package://robotarm_description/meshes/belt_arm_ros_gripper_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
- added link lower; visual mesh filename=package://robotarm_description/meshes/belt_arm_ros_lower.stl
- added link manipulator; visual mesh filename=package://robotarm_description/meshes/belt_arm_ros_manipula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
- added link upper; visual mesh filename=package://robotarm_description/meshes/belt_arm_ros_upper.stl
- added link virtualupper; visual cylinder length=0.001 radius=0.0001
Joints:
- added joint base_body: type revolute, parent base, child body, origin xyz=0 0 0.056, axis 0 0 1, limit lower=0 upper=3.2114 effort=30.0 velocity=0.5
- added joint body_lower: type revolute, parent body, child lower, origin xyz=0 0 0.074, axis 1 0 0, limit lower=0 upper=2.33874 effort=30.0 velocity=0.5
- added joint lower_virtualupper: type continuous, parent lower, child virtualupper, origin xyz=0 0 0.12, axis 1 0 0, mimic joint=body_lower multiplier=-1 offset=0
- added joint manipulator_gripper: type prismatic, parent manipulator, child gripper_left, origin xyz=0 0 0, axis 1 0 0, limit lower=0 upper=0.015 effort=30 velocity=0.5
- added joint manipulator_gripper_mimic: type prismatic, parent manipulator, child gripper_right, origin xyz=0 0 0, axis 1 0 0, limit lower=-0.015 upper=0 effort=30 velocity=0.5, mimic joint=manipulator_gripper multiplier=-1 offset=0
- added joint upper_manipulator: type continuous, parent upper, child manipulator, origin xyz=0 0.12 0, axis 1 0 0, mimic joint=virtualupper_upper multiplier=-1 offset=0
- added joint virtualupper_upper: type revolute, parent virtualupper, child upper, origin xyz=0 0 0, axis 1 0 0, limit lower=-2.24741 upper=0.484 effort=30 velocity=0.5

Commit message: debugging in progress

File: urdf/belt_robot.urdf (robot description, URDF)
Before this commit: robot robot, 8 links, 7 joints
Links:
- removed link gripper_left
- removed link gripper_right
- removed link lower
- removed link manipulator
- removed link upper
- removed link virtualupper
Joints:
- removed joint body_lower
- removed joint lower_virtualupper
- removed joint manipulator_gripper
- removed joint manipulator_gripper_mimic
- removed joint upper_manipulator
- removed joint virtualupper_upper
- joint base_body: origin xyz=0 0 0.056 -> (none)

Commit message: fixed

File: urdf/belt_robot.urdf (robot description, URDF)
Before this commit: robot robot, 2 links, 1 joints
Joints:
- joint base_body: origin (none) -> xyz=0 0 0.056

Commit message: restored

File: urdf/belt_robot.urdf (robot description, URDF)
Before this commit: robot robot, 2 links, 1 joints
Links:
- added link gripper_left; visual mesh filename=package://robotarm_description/meshes/belt_arm_ros_gripper_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
- added link gripper_right; visual mesh filename=package://robotarm_description/meshes/belt_arm_ros_gripper_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
- added link lower; visual mesh filename=package://robotarm_description/meshes/belt_arm_ros_lower.stl
- added link manipulator; visual mesh filename=package://robotarm_description/meshes/belt_arm_ros_manipula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
- added link upper; visual mesh filename=package://robotarm_description/meshes/belt_arm_ros_upper.stl
- added link virtualupper; visual cylinder length=0.001 radius=0.0001
Joints:
- added joint body_lower: type revolute, parent body, child lower, origin xyz=0 0 0.074, axis 1 0 0, limit lower=0 upper=2.33874 effort=30.0 velocity=0.5
- added joint lower_virtualupper: type continuous, parent lower, child virtualupper, origin xyz=0 0 0.12, axis 1 0 0, mimic joint=body_lower multiplier=-1 offset=0
- added joint manipulator_gripper: type prismatic, parent manipulator, child gripper_left, origin xyz=0 0 0, axis 1 0 0, limit lower=0 upper=0.015 effort=30 velocity=0.5
- added joint manipulator_gripper_mimic: type prismatic, parent manipulator, child gripper_right, origin xyz=0 0 0, axis 1 0 0, limit lower=-0.015 upper=0 effort=30 velocity=0.5, mimic joint=manipulator_gripper multiplier=-1 offset=0
- added joint upper_manipulator: type continuous, parent upper, child manipulator, origin xyz=0 0.12 0, axis 1 0 0, mimic joint=virtualupper_upper multiplier=-1 offset=0
- added joint virtualupper_upper: type revolute, parent virtualupper, child upper, origin xyz=0 0 0, axis 1 0 0, limit lower=-2.24741 upper=0.484 effort=30 velocity=0.5

Commit message: working one

File: urdf/belt_robot.urdf (robot description, URDF)
Before this commit: robot robot, 8 links, 7 joints
Joints:
- joint base_body: limit lower=0 upper=3.2114 effort=30.0 velocity=0.5 -> lower=-1 upper=1 effort=30.0 velocity=0.1
- joint body_lower: limit lower=0 upper=2.33874 effort=30.0 velocity=0.5 -> lower=4.7 upper=6 effort=30.0 velocity=0.1
- joint virtualupper_upper: limit lower=-2.24741 upper=0.484 effort=30 velocity=0.5 -> lower=-1 upper=-0.5 effort=30 velocity=0.1
